File: mosfet-fan-switch.kicad_pcb (KiCad board)
At the start: 2 copper layers, 0 parts

Commit message: Single-layer PCB for the fan driver: 56 x 44 mm, all copper on B.Cu, DRC clean
pcb/build_board.py generates the board from a part table, a track list and the
design rules, embedding the KiCad library footprints it needs. Re-running it is
a no-op: ids are derived from the content (uuid5) and the 14 electrical footprints
reuse their symbols' uuids from the sheet, so cross-probing and Update PCB from
Schematic treat the board as the same 14 parts instead of 18 unknown ones.

Home-etch rules in the .kicad_pro netclass (clearance 0.50 mm, min track 0.80 mm)
instead of KiCad's fab defaults. Result:

  Found 0 violations
  Found 0 unconnected items

56 x 44 mm (the four 3.2 mm M3 holes set the size), 18 footprints, 42 segments,
zero vias: Q2 (SOT-23) and Q3 (SO-8) sit on the copper side, which is what removes
the need for a via anywhere. /GND bus 2.0 mm along the top edge, /P12V bus 3.0 mm
along the bottom, a 1.5 mm GND return lane down the left edge, 1.5 mm /DRAIN runs.
The generator checks every net pair for crossings: no net crossings, so the 0 ohm
jumper trick was never needed.

Schematic: J1/J2/J3 connectors with (exclude_from_sim yes) - without it KiCad
exported "J1 __J1" and ngspice reads a leading J as a JFET; C3 100n and C4 10u
decoupling at the 12 V input (sim-neutral: every number in sim/run.sh is
unchanged); footprints corrected to the real packages; DNP on the model artefacts
C1, C2, L1, R6, U1, V1, V2; and a PHYSICAL PINOUTS note block, because the SPICE
symbols number MOSFET pins D-G-S while SOT-23 is 1 gate / 2 source / 3 drain, the
IRF7416 SO-8 is 1-3 source / 4 gate / 5-8 drain and the IRFZ44N TO-220 is
1 gate / 2 drain / 3 source. ERC: 0 errors, 0 warnings.

KiCad 10 behaviour that had to be pinned down before the DRC would go clean:

- A footprint's placement rotation rotates pad *positions* only; a pad's copper
  rotates only by that pad's own (at x y angle). KiCad bakes the angle into every
  pad when it places a footprint (a fresh SO-8 at (at 10 10 9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
Parts:
- added ?: MountingHole, MountingHole_3.2mm_M3, F.Cu at (2.50, 2.50)
- added ?: MountingHole, MountingHole_3.2mm_M3, F.Cu at (53.5, 2.50)
- added ?: MountingHole, MountingHole_3.2mm_M3, F.Cu at (2.50, 41.5)
- added ?: MountingHole, MountingHole_3.2mm_M3, F.Cu at (53.5, 41.5)
- added C3: 100n, C_Disc_D5.0mm_W2.5mm_P5.00mm, F.Cu at (13.0, 36.0)
- added C4: 10u, CP_Radial_D6.3mm_P2.50mm, F.Cu at (20.0, 36.0)
- added D1: 1n5819, D_DO-41_SOD81_P10.16mm_Horizontal, F.Cu at (34.0, 36.0)
- added J1: 12V IN, PinHeader_1x02_P2.54mm_Vertical, F.Cu at (9.00, 37.0)
- added J2: PWM IN, PinHeader_1x02_P2.54mm_Vertical, F.Cu at (11.0, 20.0)
- added J3: FAN OUT, PinHeader_2x03_P2.54mm_Vertical, F.Cu at (48.5, 31.1)
- added Q1: irfz44n, TO-220-3_Vertical, F.Cu at (42.0, 22.0)
- added Q2: 2n7002, SOT-23, B.Cu at (25.0, 20.0)
- added Q3: irf7416, SO-8_3.9x4.9mm_P1.27mm, B.Cu at (30.5, 21.0)
- added R1: 1k, R_Axial_DIN0207_L6.3mm_D2.5mm_P7.62mm_Horizontal, F.Cu at (14.0, 20.0)
- added R2: 10k, R_Axial_DIN0207_L6.3mm_D2.5mm_P7.62mm_Horizontal, F.Cu at (21.6, 10.6)
- added R3: 10k, R_Axial_DIN0207_L6.3mm_D2.5mm_P7.62mm_Horizontal, F.Cu at (26.0, 32.0)
- added R4: 1k, R_Axial_DIN0207_L6.3mm_D2.5mm_P7.62mm_Horizontal, F.Cu at (27.0, 12.0)
- added R5: 10k, R_Axial_DIN0207_L6.3mm_D2.5mm_P7.62mm_Horizontal, F.Cu at (38.0, 10.0)
Routing:
- net /GND: track 0.00 -> 126.4 mm
- net /P12V: track 0.00 -> 98.6 mm
- net /GATE: track 0.00 -> 22.8 mm
- net /DRAIN: track 0.00 -> 22.4 mm
- net /HIGATE: track 0.00 -> 19.1 mm
- net /LGATE: track 0.00 -> 15.9 mm
- net /BOOT: track 0.00 -> 14.5 mm
- net /PWM: track 0.00 -> 3.00 mm
Other:
- board outline added: 56 x 44 mm
- board text added: "+12V IN"
- board text added: "12V FAN DRIVER"
- board text added: "3 x 100 mA"
- board text added: "3.3V logic in"
- board text added: "D1 K +12V"
- board text added: "FAN OUT"
- board text added: "PWM IN"
- board text added: "Q1 G-D-S"
- board text added: "copper on back"
