File: mosfet-fan-switch.kicad_pcb (KiCad board)
At the start: 2 copper layers, 56 x 44 mm, 18 parts, among them J1 12V IN, J2 PWM IN, J3 FAN OUT, Q1 irfz44n, Q2 2n7002, Q3 irf7416

Commit message: pcb: grow the board to 56 x 68 mm and route the NUC interface band
The fan driver keeps its exact v1 copper (tag checkpoint-fan-driver-v1); the
NUC link lives in a new band from y=44 to y=68, below the 12 V bus.

- board 56.0 x 68.0 mm, 26 footprints, 63 track segments, zero vias
- band GND is fed from the right: the top /GND rail runs to x=51.5, drops 1.5 mm
  past the round end cap of the 12 V bus, then runs back along y=58 - so nothing
  in the band has to cross the 12 V rail
- /PWM returns to R1 through the only free corridor, the 0.8 mm lane at x=1.69
  up the left edge; JP1 (R_Axial_DIN0207 P7.62 at (5.5,14) rot 0) bridges the GND
  spine at y=14.  Fit it as a 0 ohm axial with the leads spread, or tinned wire.
- J2 pad order set for routability: 1 /PWM, 2 /GND, 3 /DEMAND, 4 /TACH_PWM; the
  schematic's J2 pin 3/4 labels were swapped to match the board.
- J4 pad order: 1 /NUC_PWM, 2 /NUC_TACH, 3 no-connect (the header's own fan
  supply), 4 /GND.  Its /GND pad sits on the band descent at x=51.62.
- silkscreen notes rewritten for the new layout (JP1 / PRO MINI / NUC FAN HEADER /
  NUC INTERFACE); labels moved clear of the reference designators.
- DRC: 0 violations, 0 unconnected pads.  Generator reports no courtyard clashes
  and no net crossings once JUMPERS covers JP1.
- gerbers, Excellon drill + map (54 hits: 0.8 x29, 1.0 x16, 1.1 x5, 3.2 x4),
  1:1 mirrored etch SVG/PDF (55.98 x 68.00 mm), both assembly PDFs, the sheet PDF
  and all three renders regenerated.
- docs/pcb-notes.md: new courtyard table, pad-to-net tables for J2/J4/JP1, the Q4
  BC547 E-B-C warning, "The NUC link" section, KiCad 10 findings (junction dots,
  Simulation_SPICE:NPN ERC, single-line .model), refreshed Known limits.
- README: NUC link section, net table rows, parts/BOM rows, wiring steps, file list.
Parts:
- added C5: 1u, CP_Radial_D8.0mm_P3.50mm, F.Cu at (16.5, 49.0)
- added C6: 100n, C_Disc_D3.8mm_W2.6mm_P2.50mm, F.Cu at (10.5, 49.0)
- added J4: NUC FAN HEADER, PinHeader_1x04_P2.54mm_Vertical, F.Cu at (44.0, 49.0)
- added JP1: R, R_Axial_DIN0207_L6.3mm_D2.5mm_P7.62mm_Horizontal, F.Cu at (5.50, 14.0)
- added Q4: BC547, TO-92_Inline_Wide, F.Cu at (40.5, 57.0)
- added R7: 10k, R_Axial_DIN0207_L6.3mm_D2.5mm_P7.62mm_Horizontal, F.Cu at (37.7, 49.0)
- added R8: 10k, R_Axial_DIN0207_L6.3mm_D2.5mm_P7.62mm_Horizontal, F.Cu at (22.5, 49.0)
- added R9: 1k, R_Axial_DIN0207_L6.3mm_D2.5mm_P7.62mm_Horizontal, F.Cu at (40.5, 44.0)
- J2: value PWM IN -> PRO MINI; footprint PinHeader_1x02_P2.54mm_Vertical -> PinHeader_1x04_P2.54mm_Vertical
- moved J2 28.8 mm to (27.0, 44.0), turned to 0 degrees
- moved ? 24.0 mm to (2.50, 65.5)
- moved ? 24.0 mm to (53.5, 65.5)
Routing:
- net /GND: track 126.4 -> 285.4 mm
- net /PWM: track 3.00 -> 62.2 mm
- net /TACH_PWM: track 0.00 -> 21.1 mm
- net /DEMAND: track 0.00 -> 19.7 mm
- net /NUC_TACH: track 0.00 -> 9.00 mm
- net /TBASE: track 0.00 -> 7.88 mm
- net /NUC_PWM: track 0.00 -> 6.30 mm
Other:
- board size 56 x 44 mm -> 56 x 68 mm
- board text added: "JP1 = 0 ohm link"
- board text added: "NUC FAN HEADER"
- board text added: "NUC INTERFACE"
- board text added: "PRO MINI"
- board text removed: "3.3V logic in"
- board text removed: "PWM IN"

Commit message: schematic: package-accurate transistor symbols; board stripped to a routing skeleton
The four transistors are now symbols whose pin numbers are the real leg numbers, so
KiCad's "symbol pin N <-> footprint pad N" rule puts every net on the correct leg and
Update PCB from Schematic agrees with the layout instead of fighting it.

- mosfet-fan-switch.kicad_sym + sym-lib-table: Q_NMOS_TO220 (1 gate, 2 drain, 3
  source), Q_NMOS_SOT23 (1 gate, 2 source, 3 drain), Q_PMOS_SO8 (1-3 source, 4 gate,
  5-8 drain), Q_NPN_TO92 (1 emitter, 2 base, 3 collector).  KiCad ships nothing like
  these: Transistor_BJT:BC547 extends Q_NPN_CBE (wrong for the flat-face TO-92) and
  there is no IRFZ44N symbol in any library at all.
- KiCad 10 ignores Sim.Pins for .model cards and writes every device line in symbol
  pin order, so the ngspice terminal order moved into .subckt wrappers in
  sim/models/*.lib:  XQ1 /GATE /DRAIN GND mos_irfz44n, XQ2 /LGATE GND /BOOT
  mos_2n7002, XQ3 /P12V x3 /BOOT /HIGATE x4 mos_irf7416, XQ4 GND /TBASE /NUC_TACH
  npn_bc547.  ngspice wants four nodes on a MOSFET card, so the bulk is spelled out
  and tied to the source inside each wrapper.
- sim/prepare_deck.py no longer repairs the NC-Q2-0 floating bulk (the three-pin
  SPICE symbols are gone); sim/variants.py and sim/nuc_link.py key the X cards and
  the pass-transistor variants now list nets in the chosen wrapper's own order.
  variants.csv is byte-identical to the pre-change baseline; fan_count.csv and
  nuc_link.csv differ only in timestep-sensitive averaged columns (supply average
  186.8 -> 187.2 mA, ITE load 40.3 -> 40.9 uA) - every DC and peak value identical.
- Q3 is drawn as the 8-pin package box, its legs tied by segmented wires with each
  node labelled once, moved east to (189.23, 170.18) so the 9.53 mm body clears the
  /BOOT branch at x=177.8.  ERC: 0 errors, 0 warnings.
- board: tools/skeleton_board.py removed the 63 generated tracks and kept all 26
  footprints, their positions and every pad's n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
Routing:
- net /GND: track 285.4 -> 0.00 mm
- net /P12V: track 98.6 -> 0.00 mm
- net /PWM: track 62.2 -> 0.00 mm
- net /GATE: track 22.8 -> 0.00 mm
- net /DRAIN: track 22.4 -> 0.00 mm
- net /TACH_PWM: track 21.1 -> 0.00 mm
- net /DEMAND: track 19.7 -> 0.00 mm
- net /HIGATE: track 19.1 -> 0.00 mm
- net /LGATE: track 15.9 -> 0.00 mm
- net /BOOT: track 14.5 -> 0.00 mm
- net /NUC_TACH: track 9.00 -> 0.00 mm
- net /TBASE: track 7.88 -> 0.00 mm
- net /NUC_PWM: track 6.30 -> 0.00 mm
Changed lines of the file:
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@@
 	(gr_line (start 2 68) (end 0 66) (stroke (width 0.1) (type solid)) (layer "Edge.Cuts"))
 	(gr_line (start 0 2) (end 2 0) (stroke (width 0.1) (type solid)) (layer "Edge.Cuts"))
-	(segment (start 5.5 3) (end 51.5 3) (width 2) (layer "B.Cu") (net 2))
-	(segment (start 9 41) (end 48.54 41) (width 3) (layer "B.Cu") (net 1))
-	(segment (start 5.5 3) (end 5.5 37) (width 1.5) (layer "B.Cu") (net 2))
-	(segment (start 9 37) (end 9 41) (width 0.8) (layer "B.Cu") (net 1))
-	(segment (start 6.46 37) (end 5.5 37) (width 0.8) (layer "B.Cu") (net 2))
-	(segment (start 13 36) (end 13 41) (width 0.8) (layer "B.Cu") (net 1))
-	(segment (start 20 36) (end 20 41) (width 0.8) (layer "B.Cu") (net 1))
-	(segment (start 13 31) (end 5.5 31) (width 0.8) (layer "B.Cu") (net 2))
-	(segment (start 20 33.5) (end 5.5 33.5) (width 0.8) (layer "B.Cu") (net 2))
-	(segment (start 27 44) (end 1.69 44) (width 0.8) (layer "B.Cu") (net 3))
-	(segment (start 1.69 44) (end 1.69 14) (width 0.8) (layer "B.Cu") (net 3))
-	(segment (start 13.12 14) (end 14 14) (width 0.8) (layer "B.Cu") (net 3))
-	(segment (start 14 14) (end 14 20) (width 0.8) (layer "B.Cu") (net 3))
-	(segment (start 21.62 20) (end 21.62 10.62) (width 0.8) (layer "B.Cu") (net 4))
-	(segment (start 21.62 20) (end 21.62 22.5) (width 0.8) (layer "B.Cu") (net 4))
-	(segment (start 21.62 22.5) (end 24.06 22.5) (width 0.8) (layer "B.Cu") (net 4))
-	(segment (start 24.06 22.5) (end 24.0625 22.5) (width 0.8) (layer "B.Cu") (net 4))
-	(segment (start 24.0625 22.5) (end 24.0625 20.95) (width 0.8) (layer "B.Cu") (net 4))
-	(segment (start 24.0625 19.05) (end 24.06 19.05) (width 0.8) (layer "B.Cu") (net 2))
-	(segment (start 24.06 19.05) (end 24.06 3) (width 0.8) (layer "B.Cu") (net 2))
-	(segment (start 25.9375 20) (end 26 20) (width 0.8) (layer "B.Cu") (net 5))
-	(segment (start 26 20) (end 26 32) (width 0.8) (layer "B.Cu") (net 5))
-	(segment (start 26 23.575) (end 28.4 23.575) (width 0.8) (layer "B.Cu") (net 5))
-	(segment (start 29.865 23.575) (end 32.405 23.575) (width 0.8) (layer "B.Cu") (net 1))
-	(segment (start 32.405 23.575) (end 32.405 41) (width 2) (layer "B.Cu") (net 1))
-	(segment (start 27 12) (end 27 16) (width 0.8) (layer "B.Cu") (net 6))
-	(segment (start 27 16) (end 32.405 16) (width 0.8) (layer "B.Cu") (net 6))
-	(segment (start 32.405 16) (end 32.405 18.425) (width 0.8) (layer "B.Cu") (net 6))
-	(segment (start 28.595 18.425) (end 28.595 16) (width 0.8) (layer "B.Cu") (net 6))
-	(segment (start 29.865 18.425) (end 29.865 16) (width 0.8) (layer "B.Cu") (net 6))
-	(segment (start 31.135 18.425) (end 31.135 16) (width 0.8) (layer "B.Cu") (net 6))
-	(segment (start 34.62 12) (end 34.62 22) (width 0.8) (layer "B.Cu") (net 7))
-	(segment (start 34.62 22) (end 42 22) (width 0.8) (layer "B.Cu") (net 7))
-	(segment (start 34.62 12) (end 38 12) (width 0.8) (layer "B.Cu") (net 7))
-	(segment (start 38 12) (end 38 10) (width 0.8) (layer "B.Cu") (net 7))
-	(segment (start 42 16.92) (end 42 3) (width 0.8) (layer "B.Cu") (net 2))
-	(segment (start 42 19.46) (end 46 19.46) (width 1.5) (layer "B.Cu") (net 8))
-	(segment (start 46 19.46) (end 46 31.08) (width 1.5) (layer "B.Cu") (net 8))
-	(segment (start 44.16 36) (end 44.16 31.08) (width 1.5) (layer "B.Cu") (net 8))
-	(segment (start 44.16 31.08) (end 46 31.08) (width 1.5) (layer "B.Cu") (net 8))
-	(segment (start 34 36) (end 34 41) (width 0.8) (layer "B.Cu") (net 1))
-	(segment (start 48.54 31.08) (end 48.54 28.54) (width 0.8) (layer "B.Cu") (net 1))
-	(segment (start 48.54 28.54) (end 48.54 26) (width 0.8) (layer "B.Cu") (net 1))
-	(segment (start 48.54 26) (end 48.54 41) (width 0.8) (layer "B.Cu") (net 1))
-	(segment (start 51.5 3) (end 51.5 58) (width 1.5) (layer "B.Cu") (net 2))
-	(segment (start 8 58) (end 51.62 58) (width 1.5) (layer "B.Cu") (net 2))
-	(segment (start 27 46.54) (end 8 46.54) (width 1.5) (layer "B.Cu") (net 2))
-	(segment (start 8 46.54) (end 8 58) (width 1.5) (layer "B.Cu") (net 2))
-	(segment (start 10.5 49) (end 30.08 49) (width 0.8) (layer "B.Cu") (net 10))
-	(segment (start 27 49.08) (end 27 49) (width 0.8) (layer "B.Cu") (net 10))
-	(segment (start 10.5 51.5) (end 10.5 58) (width 0.8) (layer "B.Cu") (net 2))
-	(segment (start 16.5 52.5) (end 16.5 58) (width 0.8) (layer "B.Cu") (net 2))
-	(segment (start 22.5 56.62) (end 22.5 58) (width 0.8) (layer "B.Cu") (net 2))
-	(segment (start 27 51.62) (end 35.5 51.62) (width 0.8) (layer "B.Cu") (net 11))
-	(segment (start 35.5 51.62) (end 35.5 44) (width 0.8) (layer "B.Cu") (net 11))
-	(segment (start 35.5 44) (end 40.5 44) (width 0.8) (layer "B.Cu") (net 11))
-	(segment (start 40.5 51.62) (end 43 51.62) (width 0.8) (layer "B.Cu") (net 12))
-	(segment (start 43 51.62) (end 43 57) (width 0.8) (layer "B.Cu") (net 12))
-	(segment (start 40.46 57) (end 40.46 58) (width 0.8) (layer "B.Cu") (net 2))
-	(segment (start 45.54 57) (end 46.54 57) (width 0.8) (layer "B.Cu") (net 13))
-	(segment (start 46.54 57) (end 46.54 49) (width 0.8) (layer "B.Cu") (net 13))
-	(segment (start 44 49) (end 37.7 49) (width 0.8) (layer "B.Cu") (net 9))
-	(segment (start 51.62 49) (end 51.62 58) (width 0.8) (layer "B.Cu") (net 2))
 	(footprint "PinHeader_1x02_P2.54mm_Vertical" (version 20260206) (generator "pcbnew") (generator_version "10.0")
 		(layer "F.Cu")

Commit message: pcb: embed the Arduino Pro Mini on sockets, grow the board to 56 x 92
- pcb/pro_mini.py: the clone hole map (35 holes) in one editable place, and the
  generator for pcb/footprints/mosfet-fan-switch.pretty/Arduino_Pro_Mini_328_Socket
- fp-lib-table so KiCad can find that footprint
- U1 sits on three female headers; pad numbers == hole numbers == symbol pins
- J5 mirrors the module's programming row for FTDI/CH340, J6 is the 2x3 ICSP
  header with pin 2 (programmer VCC) left dead on purpose
- D2 (1N5822, DO-27) and D3 (TO-220, MBR10100CT) stand unpopulated across
  /P12V-/DRAIN for the 12+ fan case
- J2 deleted; JP1 moved so its pads actually straddle the GND spine
- generated routing extended into the strip; stripped to a skeleton, DRC clean
  apart from the expected unconnected pads
Parts:
- removed J2: PRO MINI, PinHeader_1x04_P2.54mm_Vertical
- added D2: D, Diode_THT:D_DO-27_P15.24mm_Horizontal, F.Cu at (47.5, 6.00)
- added D3: TO-220-3, Package_TO_SOT_THT:TO-220-3_Vertical, F.Cu at (52.2, 30.0)
- added J5: PinHeader, Connector_PinHeader_2.54mm:PinHeader_1x06_P2.54mm_Vertical, F.Cu at (48.5, 85.7)
- added J6: PinHeader, Connector_PinHeader_2.54mm:PinHeader_2x03_P2.54mm_Vertical, F.Cu at (16.0, 62.0)
- added U1: Arduino_Pro_Mini_3V3, mosfet-fan-switch:Arduino_Pro_Mini_328_Socket, F.Cu at (14.0, 87.0)
- ? (x4): footprint MountingHole_3.2mm_M3 -> MountingHole:MountingHole_3.2mm_M3
- C3: footprint C_Disc_D5.0mm_W2.5mm_P5.00mm -> Capacitor_THT:C_Disc_D5.0mm_W2.5mm_P5.00mm
- C4: footprint CP_Radial_D6.3mm_P2.50mm -> Capacitor_THT:CP_Radial_D6.3mm_P2.50mm
- C5: footprint CP_Radial_D8.0mm_P3.50mm -> Capacitor_THT:CP_Radial_D8.0mm_P3.50mm
- C6: footprint C_Disc_D3.8mm_W2.6mm_P2.50mm -> Capacitor_THT:C_Disc_D3.8mm_W2.6mm_P2.50mm
- D1: footprint D_DO-41_SOD81_P10.16mm_Horizontal -> Diode_THT:D_DO-41_SOD81_P10.16mm_Horizontal
- J1: footprint PinHeader_1x02_P2.54mm_Vertical -> Connector_PinHeader_2.54mm:PinHeader_1x02_P2.54mm_Vertical
- J3: footprint PinHeader_2x03_P2.54mm_Vertical -> Connector_PinHeader_2.54mm:PinHeader_2x03_P2.54mm_Vertical
- J4: footprint PinHeader_1x04_P2.54mm_Vertical -> Connector_PinHeader_2.54mm:PinHeader_1x04_P2.54mm_Vertical
- JP1, R1, R2, R3, R4, R5, R7, R8, R9: footprint R_Axial_DIN0207_L6.3mm_D2.5mm_P7.62mm_Horizontal -> Resistor_THT:R_Axial_DIN0207_L6.3mm_D2.5mm_P7.62mm_Horizontal
- Q1: footprint TO-220-3_Vertical -> Package_TO_SOT_THT:TO-220-3_Vertical
- Q2: footprint SOT-23 -> Package_TO_SOT_SMD:SOT-23
- Q3: footprint SO-8_3.9x4.9mm_P1.27mm -> Package_SO:SO-8_3.9x4.9mm_P1.27mm
- Q4: footprint TO-92_Inline_Wide -> Package_TO_SOT_THT:TO-92_Inline_Wide
- moved ? 24.0 mm to (2.50, 89.5)
- moved ? 24.0 mm to (53.5, 89.5)
- moved JP1 3.50 mm to (2.00, 14.0)
Other:
- board size 56 x 68 mm -> 56 x 92 mm
- board text added: "D2 D3 spare"
- board text added: "ICSP: no 5V wire"
- board text added: "J5: 1=DTR 6=BLK"
- board text added: "PRO MINI 328 SOCKET"
- board text removed: "PRO MINI"

Commit message: sch: draw the Pro Mini itself, with its FTDI and ICSP headers
The Nano stand-in is gone.  U1 is now mosfet-fan-switch:Arduino_Pro_Mini_328,
generated from the same hole map as the board's socket footprint, so a symbol
pin number, a footprint pad number and the hole's silkscreen name are one
number.  J2 - the header that used to carry four signals to a module that was
not on the board - is deleted.

  * pcb/pro_mini.py now emits the symbol as well as the footprint.
  * tools/embed_pro_mini_schematic.py is the one-shot migration: it drops the
    Nano and J2 with their labels, no-connects and stubs, draws U1, J5 (FTDI
    row), J6 (2x3 ICSP, pin 2 deliberately dead), D2 and D3 (spare flyback
    diodes, unpopulated), and hands U1's programming-row GND to the GND rail.
  * KiCad only resolves symbols from the sheet's own lib_symbols cache, so the
    migration carries cached copies of everything it introduces.
  * Every new anchor sits on the 1.27 mm connection grid, which is what ERC's
    endpoint_off_grid check wants.
  * The board's footprints adopt the sheet's uuids, and D2/D3/J5/J6 now carry
    their real values.

ERC: 0 errors, 0 warnings.  DRC on the routing skeleton: no courtyard, silk,
clearance or hole violations; the same 7 cosmetic lib_footprint_mismatch
warnings and 68 expected unconnected pads.
Parts:
- D2: value D -> 1n5822
- D3: value TO-220-3 -> mbr10100ct
- J5: value PinHeader -> FTDI HEADER
- J6: value PinHeader -> ICSP
Changed lines of the file:
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@@
 		(at 47.5 6 -90)
 		(property "Reference" "D2" (at -2.85 0 0) (layer "F.SilkS") (effects (font (size 1 1) (thickness 0.15))))
-		(property "Value" "D" (at 0 0 0) (layer "F.Fab") (hide yes) (effects (font (size 1 1) (thickness 0.15))))
+		(property "Value" "1n5822" (at 0 0 0) (layer "F.Fab") (hide yes) (effects (font (size 1 1) (thickness 0.15))))
 		(attr through_hole)
     (fp_line (start 1.44 0) (end 2.74 0) (stroke (width 0.12) (type solid)) (layer "F.SilkS"))
@@
 		(at 52.2 30 -90)
 		(property "Reference" "D3" (at -4.11 -0.95 0) (layer "F.SilkS") (effects (font (size 1 1) (thickness 0.15))))
-		(property "Value" "TO-220-3" (at 0 0 0) (layer "F.Fab") (hide yes) (effects (font (size 1 1) (thickness 0.15))))
+		(property "Value" "mbr10100ct" (at 0 0 0) (layer "F.Fab") (hide yes) (effects (font (size 1 1) (thickness 0.15))))
 		(attr through_hole)
     (fp_line (start -2.57 -3.26) (end 7.65 -3.26) (stroke (width 0.12) (type solid)) (layer "F.SilkS"))
@@
 		(at 48.5 85.73 -180)
 		(property "Reference" "J5" (at 0 15.87 0) (layer "F.SilkS") (effects (font (size 1 1) (thickness 0.15))))
-		(property "Value" "PinHeader" (at 0 0 0) (layer "F.Fab") (hide yes) (effects (font (size 1 1) (thickness 0.15))))
+		(property "Value" "FTDI HEADER" (at 0 0 0) (layer "F.Fab") (hide yes) (effects (font (size 1 1) (thickness 0.15))))
 		(attr through_hole)
     (fp_line (start -1.38 -1.38) (end 0 -1.38) (stroke (width 0.12) (type solid)) (layer "F.SilkS"))
@@
 		(at 16 62 0)
 		(property "Reference" "J6" (at 1.275 -3.17 0) (layer "F.SilkS") (effects (font (size 1 1) (thickness 0.15))))
-		(property "Value" "PinHeader" (at 0 0 0) (layer "F.Fab") (hide yes) (effects (font (size 1 1) (thickness 0.15))))
+		(property "Value" "ICSP" (at 0 0 0) (layer "F.Fab") (hide yes) (effects (font (size 1 1) (thickness 0.15))))
 		(attr through_hole)
     (fp_line (start -1.38 -1.38) (end 0 -1.38) (stroke (width 0.12) (type solid)) (layer "F.SilkS"))
