File: fan-switch-booster/mosfet-fan-switch.kicad_sch (KiCad schematic)
At the start: 35 parts, among them J1 12V IN, J3 FAN OUT, J4 NUC FAN HEADER, J5 FTDI HEADER, J6 ICSP, Q1 irfz44n, Q2 2n7002, Q3 irf7416, Q4 BC547, U1 Arduino_Pro_Mini_3V3

Commit message: pcb done
Parts:
- removed J6: ICSP, Connector_PinHeader_2.54mm:PinHeader_2x03_P2.54mm_Vertical, symbol Connector_Generic:Conn_02x03_Odd_Even
Connections:
- net GND: now also U1.14 (GND)
- net MISO: no longer names the net of U1.22 (D12)
- net MOSI: no longer names the net of U1.23 (D11)
- net SCK: no longer names the net of U1.21 (D13)
- no-connect marks 19 -> 21
Changed lines of the file:
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@@
 	)
 	(no_connect
-		(at 80.01 139.7)
-	)
-	(no_connect
 		(at 44.45 138.43)
 	)
@@
 		)
 	)
-	(label "SCK"
-		(at 22.86 121.92 180)
-		(effects
-			(font
-				(size 1.27 1.27)
-			)
-			(justify right bottom)
-		)
-	)
 	(label "GND"
 		(at 400.05 177.8 270)
@@
 		)
 	)
-	(label "GND"
-		(at 35.56 124.46 0)
-		(effects
-			(font
-				(size 1.27 1.27)
-			)
-			(justify left bottom)
-		)
-	)
 	(label "BLK"
 		(at 22.86 166.37 180)
@@
 		)
 	)
-	(label "MOSI"
-		(at 80.01 162.56 0)
-		(effects
-			(font
-				(size 1.27 1.27)
-			)
-			(justify left bottom)
-		)
-	)
 	(label "DRAIN"
 		(at 246.38 175.26 180)
@@
 		)
 	)
+	(label "GND"
+		(at 80.01 139.7 0)
+		(effects
+			(font
+				(size 1.27 1.27)
+			)
+			(justify left bottom)
+		)
+	)
 	(label "DRAIN"
 		(at 261.62 175.26 0)
@@
 		)
 	)
-	(label "SCK"
-		(at 80.01 157.48 0)
-		(effects
-			(font
-				(size 1.27 1.27)
-			)
-			(justify left bottom)
-		)
-	)
 	(label "GND"
 		(at 44.45 146.05 180)
@@
 		)
 	)
-	(label "RST"
-		(at 22.86 124.46 180)
-		(effects
-			(font
-				(size 1.27 1.27)
-			)
-			(justify right bottom)
-		)
-	)
-	(label "MOSI"
-		(at 35.56 121.92 0)
-		(effects
-			(font
-				(size 1.27 1.27)
-			)
-			(justify left bottom)
-		)
-	)
 	(label "GND"
 		(at 307.34 198.12 180)
@@
 		)
 	)
-	(label "MISO"
-		(at 22.86 119.38 180)
-		(effects
-			(font
-				(size 1.27 1.27)
-			)
-			(justify right bottom)
-		)
-	)
 	(label "GND"
 		(at 330.2 227.33 270)
@@
 		)
 	)
-	(label "MISO"
-		(at 80.01 160.02 0)
-		(effects
-			(font
-				(size 1.27 1.27)
-			)
-			(justify left bottom)
-		)
-	)
 	(symbol
 		(lib_id "Simulation_SPICE:VPULSE")
@@
 		)
 	)
-	(symbol
-		(lib_id "Connector_Generic:Conn_02x03_Odd_Even")
-		(at 27.94 121.92 0)
-		(unit 1)
-		(body_style 1)
-		(exclude_from_sim yes)
-		(in_bom yes)
-		(on_board yes)
-		(in_pos_files yes)
-		(dnp no)
-		(property "Reference" "J6"
-			(at 27.94 127 0)
-			(show_name no)
-			(do_not_autoplace no)
-			(effects
-				(font
-					(size 1.27 1.27)
-				)
-			)
-		)
-		(property "Value" "ICSP"
-			(at 27.94 116.84 0)
-			(show_name no)
-			(do_not_autoplace no)
-			(effects
-				(font
-					(size 1.27 1.27)
-				)
-			)
-		)
-		(property "Footprint" "Connector_PinHeader_2.54mm:PinHeader_2x03_P2.54mm_Vertical"
-			(at 27.94 121.92 0)
-			(hide yes)
-			(show_name no)
-			(do_not_autoplace no)
-			(effects
-				(font
-					(size 1.27 1.27)
-				)
-			)
-		)
-		(property "Datasheet" ""
-			(at 27.94 121.92 0)
-			(hide yes)
-			(show_name no)
-			(do_not_autoplace no)
-			(effects
-				(font
-					(size 1.27 1.27)
-				)
-			)
-		)
-		(property "Description" "Generic connector, double row, 02x03, odd/even numbering"
-			(at 27.94 121.92 0)
-			(hide yes)
-			(show_name no)
-			(do_not_autoplace no)
-			(effects
-				(font
-					(size 1.27 1.27)
-				)
-			)
-		)
-		(property "Note" "program the 328 with another Arduino over five wires: pin 2 is the programmer's 5 V and must stay unconnected on a 3.3 V board"
-			(at 27.94 121.92 0)
-			(hide yes)
-			(show_name no)
-			(do_not_autoplace no)
-			(effects
-				(font
-					(size 1.27 1.27)
-				)
-			)
-		)
-		(pin "1"
-		)
-		(pin "2"
-		)
-		(pin "3"
-		)
-		(pin "4"
-		)
-		(pin "5"
-		)
-		(pin "6"
-		)
-		(instances
-			(project "mosfet-fan-switch"
-				(path "/70af4f7e-8b7a-484f-96e0-6ca2b9e2231e"
-					(reference "J6")
-					(unit 1)
-				)
-			)
-		)
+	(no_connect
+		(at 80.00999999999999 157.48)
+	)
+	(no_connect
+		(at 80.00999999999999 160.02)
+	)
+	(no_connect
+		(at 80.00999999999999 162.56)
 	)
 	(sheet_instances

Commit message: pcb manually designed
Connections:
- no-connect marks 21 -> 20
Changed lines of the file:
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@@
 		)
 	)
-	(text "PHYSICAL PINOUTS - symbols use package pin order: sheet numbers = board legs\nQ2  2N7002  SOT-23    1 gate /LGATE    2 source /GND     3 drain /BOOT\nQ3  IRF7416 SO-8      1,2,3 source /P12V   4 gate /BOOT   5..8 drain /HIGATE\nQ1  IRFZ44N TO-220    1 gate /GATE     2 drain /DRAIN    3 source /GND\nQ4  BC547   TO-92     1 emitter /GND   2 base /TBASE     3 collector /NUC_TACH\nD1  1N5819  DO-41     banded end (cathode) to +12 V, other end to /DRAIN\nJ3  3 fans            odd pins = +12 V, even pins = the switched /DRAIN side\nngspice's own order (D-G-S-B, C-B-E) lives in the sim/models/ subckt wrappers\nJ5  FTDI    1 DTR  2 TX0  3 RX1  4 P3V3  5 GND  6 BLK\nJ6  ICSP    1 MISO 3 SCK  4 MOSI 5 RST  6 GND   (pin 2 stays dead)\nU1  35 module holes: symbol pin number = socket pad number\ndocs/pcb-notes.md carries the full pad-to-net table for the board."
+	(text "PHYSICAL PINOUTS - symbols use package pin order: sheet numbers = board legs\nQ2  2N7002  SOT-23    1 gate /LGATE    2 source /GND     3 drain /BOOT\nQ3  IRF7416 SO-8      1,2,3 source /P12V   4 gate /BOOT   5..8 drain /HIGATE\nQ1  IRFZ44N TO-220    1 gate /GATE     2 drain /DRAIN    3 source /GND\nQ4  BC547   TO-92     1 emitter /GND   2 base /TBASE     3 collector /NUC_TACH\nD1  1N5819  DO-41     banded end (cathode) to +12 V, other end to /DRAIN\nJ3  3 fans            odd pins = +12 V, even pins = the switched /DRAIN side\nngspice's own order (D-G-S-B, C-B-E) lives in the sim/models/ subckt wrappers\nJ5  FTDI    1 DTR  2 TX0  3 RX1  4 P3V3  5 GND  6 BLK   (no ICSP header on this board)\nU1  35 module holes: symbol pin number = socket pad number\ndocs/pcb-notes.md carries the full pad-to-net table for the board."
 		(exclude_from_sim no)
 		(at 155 250 0)
@@
 	)
 	(no_connect
-		(at 35.56 119.38)
-	)
-	(no_connect

Commit message: sch: drop J6, land U1 pad 14 on GND, add four M3 mounting holes
Parts:
- added MK1, MK2, MK3, MK4: M3 mounting hole, MountingHole:MountingHole_3.2mm_M3, symbol Mechanical:MountingHole
